File: deska.brd (EAGLE design)
At the start: 25.7 x 40 mm, 11 parts

Commit message: deska;
Parts:
- R2: value 68k -> 1k
- renumbered 230V to 5V
Changed lines of the file:
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@@
 <?xml version="1.0" encoding="utf-8"?>
 <!DOCTYPE eagle SYSTEM "eagle.dtd">
-<eagle version="7.7.0">
+<eagle version="9.1.3">
 <drawing>
 <settings>
 <setting alwaysvectorfont="no"/>
+<setting keepoldvectorfont="yes"/>
 <setting verticaltext="up"/>
 </settings>
@@
 <param name="dpMaxLengthDifference" value="10mm"/>
 <param name="dpGapFactor" value="2.5"/>
-<param name="checkGrid" value="0"/>
 <param name="checkAngle" value="0"/>
 <param name="checkFont" value="1"/>
 <param name="checkRestrict" value="1"/>
+<param name="checkStop" value="0"/>
+<param name="checkValues" value="0"/>
+<param name="checkNames" value="1"/>
+<param name="checkWireStubs" value="1"/>
+<param name="checkPolygonWidth" value="0"/>
 <param name="useDiameter" value="13"/>
 <param name="maxErrors" value="50"/>
@@
 </autorouter>
 <elements>
-<element name="230V" library="con-amp-quick" package="02P" value="" x="8.255" y="2.54">
+<element name="5V" library="con-amp-quick" package="02P" value="" x="8.255" y="2.54">
+<attribute name="MF" value="" x="8.255" y="2.54" size="1.778" layer="27" display="off"/>
 <attribute name="MPN" value="" x="8.255" y="2.54" size="1.778" layer="27" display="off"/>
-<attribute name="MF" value="" x="8.255" y="2.54" size="1.778" layer="27" display="off"/>
+<attribute name="OC_FARNELL" value="unknown" x="8.255" y="2.54" size="1.778" layer="27" display="off"/>
 <attribute name="OC_NEWARK" value="unknown" x="8.255" y="2.54" size="1.778" layer="27" display="off"/>
-<attribute name="OC_FARNELL" value="unknown" x="8.255" y="2.54" size="1.778" layer="27" display="off"/>
 </element>
 <element name="D1" library="diode" package="DO41-10" value="1N4004" x="12.065" y="7.62"/>
 <element name="DETECT" library="led" package="LED3MM" value="" x="17.145" y="22.225" rot="R180"/>
 <element name="NAPAJENI" library="con-amp-quick" package="02P" value="" x="15.875" y="2.54">
+<attribute name="MF" value="" x="15.875" y="2.54" size="1.778" layer="27" display="off"/>
 <attribute name="MPN" value="" x="15.875" y="2.54" size="1.778" layer="27" display="off"/>
-<attribute name="MF" value="" x="15.875" y="2.54" size="1.778" layer="27" display="off"/>
+<attribute name="OC_FARNELL" value="unknown" x="15.875" y="2.54" size="1.778" layer="27" display="off"/>
 <attribute name="OC_NEWARK" value="unknown" x="15.875" y="2.54" size="1.778" layer="27" display="off"/>
-<attribute name="OC_FARNELL" value="unknown" x="15.875" y="2.54" size="1.778" layer="27" display="off"/>
 </element>
 <element name="OK1" library="optocoupler" package="DIL04" value="PC817" x="12.065" y="19.05">
+<attribute name="MF" value="" x="12.065" y="19.05" size="1.778" layer="27" display="off"/>
 <attribute name="MPN" value="PC817X4J000F" x="12.065" y="19.05" size="1.778" layer="27" display="off"/>
-<attribute name="MF" value="" x="12.065" y="19.05" size="1.778" layer="27" display="off"/>
+<attribute name="OC_FARNELL" value="9707727" x="12.065" y="19.05" size="1.778" layer="27" display="off"/>
 <attribute name="OC_NEWARK" value="97K7059" x="12.065" y="19.05" size="1.778" layer="27" display="off"/>
-<attribute name="OC_FARNELL" value="9707727" x="12.065" y="19.05" size="1.778" layer="27" display="off"/>
 </element>
-<element name="R2" library="resistor" package="0207/7" value="68k" x="12.065" y="11.43"/>
+<element name="R2" library="resistor" package="0207/7" value="1k" x="12.065" y="11.43"/>
 <element name="R3" library="resistor" package="0207/7" value="10k" x="12.065" y="33.02"/>
 <element name="R4" library="resistor" package="0207/7" value="1k" x="12.065" y="38.1"/>
@@
 </signal>
 <signal name="N$3">
-<contactref element="230V" pad="2"/>
+<contactref element="5V" pad="2"/>
 <contactref element="R2" pad="1"/>
 <wire x1="9.525" y1="2.54" x2="9.525" y2="10.16" width="0.8128" layer="16"/>
@@
 </signal>
 <signal name="N$4">
-<contactref element="230V" pad="1"/>
+<contactref element="5V" pad="1"/>
 <contactref element="D1" pad="C"/>
 <wire x1="6.985" y1="2.54" x2="6.985" y2="7.62" width="0.8128" layer="16"/>
@@
 </signal>
 </signals>
+<mfgpreviewcolors>
+<mfgpreviewcolor name="soldermaskcolor" color="0xC8008000"/>
+<mfgpreviewcolor name="silkscreencolor" color="0xFFFEFEFE"/>
+<mfgpreviewcolor name="backgroundcolor" color="0xFF282828"/>
+<mfgpreviewcolor name="coppercolor" color="0xFFFFBF00"/>
+<mfgpreviewcolor name="substratecolor" color="0xFF786E46"/>
+</mfgpreviewcolors>
 </board>
 </drawing>

Commit message: v0.3
Parts:
- removed D1: 1N4004, diode:DO41-10
- R4: value 1k -> 220
Connections:
- removed net N$4: 5V.1, D1.C
- net N$6: now also 5V.1; no longer D1.A
Routing:
- net N$4: track 5.08 -> 0.00 mm
- net N$6: track 9.94 -> 8.67 mm
Changed lines of the file:
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@@
 <attribute name="OC_NEWARK" value="unknown" x="8.255" y="2.54" size="1.778" layer="27" display="off"/>
 </element>
-<element name="D1" library="diode" package="DO41-10" value="1N4004" x="12.065" y="7.62"/>
 <element name="DETECT" library="led" package="LED3MM" value="" x="17.145" y="22.225" rot="R180"/>
 <element name="NAPAJENI" library="con-amp-quick" package="02P" value="" x="15.875" y="2.54">
@@
 <element name="R2" library="resistor" package="0207/7" value="1k" x="12.065" y="11.43"/>
 <element name="R3" library="resistor" package="0207/7" value="10k" x="12.065" y="33.02"/>
-<element name="R4" library="resistor" package="0207/7" value="1k" x="12.065" y="38.1"/>
+<element name="R4" library="resistor" package="0207/7" value="220" x="12.065" y="38.1"/>
 <element name="R5" library="resistor" package="0207/7" value="1k" x="12.065" y="35.56" rot="R180"/>
 <element name="STATUS" library="led" package="LED3MM" value="" x="5.715" y="22.225"/>
@@
 <wire x1="9.525" y1="2.54" x2="9.525" y2="10.16" width="0.8128" layer="16"/>
 <wire x1="9.525" y1="10.16" x2="8.255" y2="11.43" width="0.8128" layer="16"/>
-</signal>
-<signal name="N$4">
-<contactref element="5V" pad="1"/>
-<contactref element="D1" pad="C"/>
-<wire x1="6.985" y1="2.54" x2="6.985" y2="7.62" width="0.8128" layer="16"/>
 </signal>
 <signal name="GND">
@@
 <signal name="N$6">
 <contactref element="OK1" pad="2"/>
-<contactref element="D1" pad="A"/>
-<wire x1="13.335" y1="15.24" x2="13.335" y2="10.16" width="0.8128" layer="16"/>
-<wire x1="13.335" y1="10.16" x2="15.875" y2="7.62" width="0.8128" layer="16"/>
-<wire x1="15.875" y1="7.62" x2="17.145" y2="7.62" width="0.8128" layer="16"/>
+<wire x1="14.605" y1="13.97" x2="14.605" y2="8.89" width="0.8128" layer="16"/>
+<wire x1="14.605" y1="8.89" x2="15.875" y2="7.62" width="0.8128" layer="16"/>
+<contactref element="5V" pad="1"/>
+<wire x1="6.985" y1="2.54" x2="14.605" y2="8.89" width="0" layer="19" extent="16-16"/>
+<wire x1="13.335" y1="15.24" x2="14.605" y2="13.97" width="0.8128" layer="16"/>
 </signal>
 </signals>
